File: MAN_Motor_Drivers/MAN_Motor_Drivers.kicad_pcb (KiCad board)
At the start: 2 copper layers, 47.2 x 78 mm, 53 parts, among them J1 Conn_01x05, J10 VIN, J11 Conn_01x05, J12 Conn_01x05, J13 Conn_01x05, J14 Conn_01x02, J2 Conn_01x05, J3 Conn_01x05, J4 MOTOR1_OUT1, J5 MOTOR3_OUT1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

Commit message: current version
Parts:
- added C22: CP, Capacitor_SMD:CP_Elec_8x10, F.Cu at (167.8, 37.8)
- added D2: LED, LED_SMD:LED_0603_1608Metric_Pad1.05x0.95mm_HandSolder, F.Cu at (170.0, 57.2)
- added D3: LED, LED_SMD:LED_0603_1608Metric_Pad1.05x0.95mm_HandSolder, F.Cu at (169.2, 80.5)
- added D4: LED, LED_SMD:LED_0603_1608Metric_Pad1.05x0.95mm_HandSolder, F.Cu at (169.2, 104.0)
- added H1: MountingHole, MountingHole:MountingHole_2.7mm_M2.5, F.Cu at (138.8, 22.5)
- added H2: MountingHole, MountingHole:MountingHole_2.7mm_M2.5, F.Cu at (177.5, 106.2)
- added R13: 1k, Resistor_SMD:R_0603_1608Metric_Pad1.05x0.95mm_HandSolder, F.Cu at (170.0, 55.2)
- added R14: 1k, Resistor_SMD:R_0603_1608Metric_Pad1.05x0.95mm_HandSolder, F.Cu at (169.2, 78.8)
- added R15: 1k, Resistor_SMD:R_0603_1608Metric_Pad1.05x0.95mm_HandSolder, F.Cu at (169.2, 102.2)
- added U7: DPST_ON_OFF, Button_Switch_THT:DPST_ON_OFF, F.Cu at (166.8, 27.0)
- moved J10 32.5 mm to (145.0, 29.8), turned to 90 degrees
- moved C13 0.79 mm to (174.2, 45.2), turned to 270 degrees
- moved J14 0.56 mm to (138.5, 36.0), turned to 180 degrees
- moved C14 0.50 mm to (173.8, 68.2), turned to 270 degrees
- moved C15 0.25 mm to (173.8, 92.0), turned to 270 degrees
Connections:
- C13 pad 1: /VIN -> Net-(C13-Pad1)
- C14 pad 1: /VIN -> Net-(C13-Pad1)
- C15 pad 1: /VIN -> Net-(C13-Pad1)
- U1 pad 17: (no net) -> GND
- U2 pad 17: (no net) -> GND
- U3 pad 17: (no net) -> GND
- U4 pad 1: /VIN -> Net-(C13-Pad1)
- U5 pad 1: /VIN -> Net-(C13-Pad1)
- U6 pad 1: /VIN -> Net-(C13-Pad1)
Routing:
- net Net-(C13-Pad1): track 0.00 -> 84.3 mm
- net /VIN: track 81.4 -> 0.00 mm
- net +12V: track 92.1 -> 106.0 mm
- net GND: track 0.00 -> 3.85 mm
- net Net-(D2-Pad2): track 0.00 -> 2.00 mm
- net /OUT2_A: track 4.07 -> 2.26 mm
- net Net-(D4-Pad2): track 0.00 -> 1.75 mm
- net Net-(D3-Pad2): track 0.00 -> 1.75 mm
- net +3V3: track 89.6 -> 90.9 mm
- added copper zone on F.Cu, net /VIN
- added copper zone on F.Cu, net Net-(C13-Pad1)
Other:
- board size 47.2 x 78 mm -> 47.2 x 91.8 mm
- rule pad_to_mask_clearance: 0.051 -> 0.1
- board text added: "MANIPULATOR M4P v1.0"
