File: MAN_Motor_Drivers/MAN_Motor_Drivers.sch (KiCad schematic (older format))
At the start: 53 parts, among them J1 Conn_01x05, J10 VIN, J11 Conn_01x05, J12 Conn_01x05, J13 Conn_01x05, J14 Conn_01x02, J2 Conn_01x05, J3 Conn_01x05, J4 MOTOR1_OUT1, J5 MOTOR3_OUT1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

Commit message: current version
Parts:
- added C22: CP, Capacitor_SMD:CP_Elec_8x10, symbol Device:CP
- added D2, D3, D4: LED, LED_SMD:LED_0603_1608Metric_Pad1.05x0.95mm_HandSolder, symbol Device:LED
- added H1, H2: MountingHole, MountingHole:MountingHole_2.7mm_M2.5, symbol Mechanical:MountingHole
- added R13, R14, R15: 1k, Resistor_SMD:R_0603_1608Metric_Pad1.05x0.95mm_HandSolder, symbol Device:R
- added U7: DPST_ON_OFF, Button_Switch_THT:DPST_ON_OFF, symbol Switches:DPST_ON_OFF
Connections:
- net +12V: now also R13.2, R14.2, R15.2
- net GND: now also U1.17 (PADGND), U2.17 (PADGND), U3.17 (PADGND), C22.2, D2.1 (K), D3.1 (K), D4.1 (K)
- net VIN: now also U7.1 (IN); no longer C13.1, C14.1, C15.1, U4.1 (VI), U5.1 (VI), U6.1 (VI)
- new net: C13.1, C14.1, C15.1, C22.1, U4.1 (VI), U5.1 (VI), U6.1 (VI), U7.2 (OUT)
- new net: D2.2 (A), R13.1
- new net: D3.2 (A), R14.1
- new net: D4.2 (A), R15.1
- no-connect marks 12 -> 13
Other:
- moved on the sheet: C13, C14, C15, C16, C17, C18, J10, U4, U5, U6
